File: pcb/Stoplight.kicad_sch (KiCad schematic)
At the start: 16 parts, among them IC1 ATtiny85-20M, IC2 AP7375-33SA-7

Commit message: Good double-sided design
Parts:
- R1, R2, R3, R4: footprint Resistor_SMD:R_0201_0603Metric -> Resistor_SMD:R_0603_1608Metric
Changed lines of the file:
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@@
 			)
 		)
-		(property "Footprint" "Resistor_SMD:R_0201_0603Metric"
+		(property "Footprint" "Resistor_SMD:R_0603_1608Metric"
 			(at 78.74 34.798 90)
 			(effects
@@
 			)
 		)
-		(property "Footprint" "Resistor_SMD:R_0201_0603Metric"
+		(property "Footprint" "Resistor_SMD:R_0603_1608Metric"
 			(at 91.44 34.798 90)
 			(effects
@@
 			)
 		)
-		(property "Footprint" "Resistor_SMD:R_0201_0603Metric"
+		(property "Footprint" "Resistor_SMD:R_0603_1608Metric"
 			(at 114.3 147.828 90)
 			(effects
@@
 			)
 		)
-		(property "Footprint" "Resistor_SMD:R_0201_0603Metric"
+		(property "Footprint" "Resistor_SMD:R_0603_1608Metric"
 			(at 114.3 152.908 90)
 			(effects

Commit message: Another solid design, but going to try for even simpler
Parts:
- added POT1: TC33X-2-103E, digikey-footprints:Trimpot_3.8mmx3.6mm_TC33X-2-103E, symbol dk_Trimmer-Potentiometers:TC33X-2-103E
- added TP8: RST, Connector_PinHeader_1.00mm:PinHeader_1x01_P1.00mm_Vertical, symbol Connector:TestPoint
Connections:
- net +5V: now also POT1.1 (CCW)
- net GND: now also POT1.3 (CW)
- net RST: now also TP8.1
- net LED_G: no longer names the net of IC1.5 (XTAL2/PB4)
- net LED_G: no longer R4.2
- net LED_R renamed DIM
- net DIM: now also POT1.2 (Wiper); no longer R3.2
- net MISO renamed MISO/G
- net MISO/G: now also R4.2
- net MOSI renamed MOSI/R
- net MOSI/R: now also R3.2
- net SCK/A1 renamed SCK/BATT

Commit message: Almost entirely single-layer now
Connections:
- net MISO/G: now also R3.2; no longer R4.2
- net MOSI/R: now also R4.2; no longer R3.2
Changed lines of the file:
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@@
 	(global_label "MISO{slash}G"
 		(shape input)
-		(at 119.38 151.13 0)
+		(at 119.38 146.05 0)
 		(fields_autoplaced yes)
 		(effects
@@
 		)
 		(property "Intersheetrefs" "${INTERSHEET_REFS}"
-			(at 129.5619 151.13 0)
+			(at 129.5619 146.05 0)
 			(effects
 				(font
@@
 	(global_label "MOSI{slash}R"
 		(shape input)
-		(at 119.38 146.05 0)
+		(at 119.38 151.13 0)
 		(fields_autoplaced yes)
 		(effects
@@
 		)
 		(property "Intersheetrefs" "${INTERSHEET_REFS}"
-			(at 129.5619 146.05 0)
+			(at 129.5619 151.13 0)
 			(effects
 				(font

Commit message: Swapped mcu package to SOIC-8 for easier soldering
Parts:
- D1: Part Number (none) -> WP59SURKZGW; URL (none) -> https://www.digikey.com/en/products/detail/kingbright/WP59S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
- IC1: footprint Package_DFN_QFN:QFN-20-1EP_4x4mm_P0.5mm_EP2.6x2.6mm -> digikey-footprints:SOIC-8_W5.3mm; symbol MCU_Microchip_ATtiny:ATtiny85-20M -> dk_Embedded-Microcontrollers:ATTINY85-20SU; Category (none) -> Integrated Circuits (ICs); DK_Datasheet_Link (none) -> http://www.microchip.com/mymicrochip/filehandler.aspx?ddocn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; DK_Detail_Page (none) -> /product-detail/en/microchip-technology/ATTINY85-20SU/ATTIN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; Family (none) -> Embedded - Microcontrollers; MPN (none) -> ATTINY85-20SU; Manufacturer (none) -> Microchip Technology; Status (none) -> Active
- IC2: value AP7375-33SA-7 -> AP7375-50SA-7; footprint AP7375-33SA-7:SOT96P240X110-3N -> AP7375-50SA-7; Part Number AP7375-33SA-7 -> AP7375-50SA-7; URL https://www.digikey.com/en/products/detail/diodes-incorporated/AP7375-33SA-7/16400213?s=N4IgTCBcDaIIIAUDsBmJBWAtClBlOmSIAugL5A -> https://www.digikey.com/en/products/detail/diodes-incorporated/AP7375-50SA-7/16400218?s=N4IgjCBcpgbFoDGUBmBDANgZwKYBoQB7KAbRABYwBmKsADhAF0CAHAFyhAGU2AnASwB2AcxABfApQQhkkdNnxFSIKuQDs5Wk1YdI3PkNESQsAJzTZ83AWKQy5AAymqz7SHaceAkeIIAmAFY-C1RMayU7ED8wP3I6CGZ3XX1vI38AgJC5MMVbMio6Uwcwc0SPPS9DXxAAtSosq1zlPxaaBJ1PAx9jMAdYTOgZUIUbZXakzgARQgBXACMMHGqY0whByxzRyMcAx1KOiq608HI-c3Xh8LzwN3KUqp61NXOkS6bI2NW1cbvK7oJ6HQHA1NhF8lQAnQIbdkn9jiUniCRmCbmVYUdlqZCkirspgYxjH4%2BvALtlkdcCn46OoYZ1UtU-GoHMDSY0tmQfuj6cYALRrV5k3GRLQEgg88g494c2KtJi8gYCtkoiD%2BED%2BTRysVqSXskDfNR0eJ4EViU1AA
- R1: value 10K -> 10K .1%; Part Number ERJ-1GNF64R9C -> ERA-1AEB103C; URL https://www.digikey.com/en/products/detail/panasonic-electronic-components/ERJ-1GNF64R9C/2035977 -> https://www.digikey.com/en/products/detail/panasonic-electronic-components/ERA-1AEB103C/5035568
- R2: value 3K3 -> 3K3 0.1%; Part Number ERJ-1GNF64R9C -> ERA-1AEB332C; URL https://www.digikey.com/en/products/detail/panasonic-electronic-components/ERJ-1GNF64R9C/2035977 -> https://www.digikey.com/en/products/detail/panasonic-electronic-components/ERA-1AEB332C/13149156?s=N4IgjCBcoExaBjKAzAhgGwM4FMA0IB7KAbRAHYBWGAFhAF18AHAFyhAGVmAnASwDsA5iAC%2B%2BAMzwQSSGix5CJcmIgMQLNp16CR%2BCpOmyc%2BIpFLKAbAE4wtVesgdu-IaPDn9KDEYWmQYywAMZAAc9EysDprOOuBkHjJe8iakMAFgenYRjlou%2BNTu0FKecsaKFNTpYWpZUdquYGS0hQaJpb4VDebumRpOdfgwVPGGSYo0MJZituG9OTFkQcOtPqQqM5F9ueBgMHHNxd7JIHA9DgAiBACuAEbo2DE71kslK36BZHGn2dH1FAEBz0OinyFE%2B62%2B-XAFGUgNGvjW1VmP3wYEswUssLapABdFcqWCen2CReRzEADoxAACADWAHkABYAW0wVXsIAAqnweMxacgALLYVCYS5ce6uAC0ECJIyx4BxEqaiAOcNI%2BX%2B8vw4sJSuJQPhIAGBuO1AkuM1ex1Mte5gClkmZFwYHlwmEQA
Connections:
- net +5V: now also IC1.8 (VCC); no longer IC1.15 (VCC)
- net GND: now also IC1.4 (GND); no longer IC1.21 (GND), IC1.8 (GND)
- net MISO/G: now also IC1.6 (PB1); no longer IC1.12 (PB1)
- net MOSI/R: now also IC1.5 (PB0); no longer IC1.11 (AREF/PB0)
- net SCK/BATT: now also IC1.7 (PB2); no longer IC1.14 (PB2)
Other:
- moved on the sheet: IC1

Commit message: Ordered v1, updated part numbers to reflect availability
Parts:
- C13: Part Number GRM158R61A226ME15D -> GMC04X5R226M10NT; URL https://www.digikey.com/en/products/detail/murata-electroni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 -> https://www.digikey.com/en/products/detail/cal-chip-electro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
- C4: value 2.2uF,100V -> 2.2uF, 50V; URL https://www.digikey.com/en/products/detail/tdk-corporation/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 -> https://www.digikey.com/en/products/detail/taiyo-yuden/UMK2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
- POT1: DK_Detail_Page /product-detail/en/bourns-inc/TC33X-2-103E/TC33X-103ETR-ND/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 -> (none)
- R3: value 65 -> 150; Part Number ERJ-1GNF64R9C -> ERA-3AEB151V; URL https://www.digikey.com/en/products/detail/panasonic-electronic-components/ERJ-1GNF64R9C/2035977 -> https://www.digikey.com/en/products/detail/panasonic-electronic-components/ERA-3AEB151V/1465834
- R4: value 65 -> 85; Part Number ERJ-1GNF64R9C -> ERJ-3EKF84R5V; URL https://www.digikey.com/en/products/detail/panasonic-electronic-components/ERJ-1GNF64R9C/2035977 -> https://www.digikey.com/en/products/detail/panasonic-electronic-components/ERJ-3EKF84R5V/196495
Changed lines of the file:
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@@
 			)
 		)
-		(property "Value" "2.2uF,100V"
+		(property "Value" "2.2uF, 50V"
 			(at 204.47 48.2599 0)
 			(effects
@@
 			)
 		)
-		(property "URL" "https://www.digikey.com/en/products/detail/tdk-corporation/C2012X7R2A225K125AC/20482638"
+		(property "URL" "https://www.digikey.com/en/products/detail/taiyo-yuden/UMK212BB7225KG-T/3194965"
 			(at 200.66 46.99 0)
 			(effects
@@
 			)
 		)
-		(property "Part Number" "GRM158R61A226ME15D"
+		(property "Part Number" "GMC04X5R226M10NT"
 			(at 261.62 52.07 0)
 			(effects
@@
 			)
 		)
-		(property "URL" "https://www.digikey.com/en/products/detail/murata-electronics/GRM158R61A226ME15D/16033379"
+		(property "URL" "https://www.digikey.com/en/products/detail/cal-chip-electronics-inc/GMC04X5R226M10NT/23571654"
 			(at 261.62 52.07 0)
 			(effects
@@
 			)
 		)
-		(property "DK_Detail_Page" "/product-detail/en/bourns-inc/TC33X-2-103E/TC33X-103ETR-ND/612858"
-			(at 137.16 83.82 0)
-			(effects
-				(font
-					(size 1.524 1.524)
-				)
-				(justify left)
-				(hide yes)
-			)
-		)
 		(property "Manufacturer" "Bourns Inc."
 			(at 137.16 78.74 0)
@@
 			)
 		)
-		(property "Value" "65"
+		(property "Value" "150"
 			(at 114.3 142.24 90)
 			(effects
@@
 			)
 		)
-		(property "Part Number" "ERJ-1GNF64R9C"
+		(property "Part Number" "ERA-3AEB151V"
 			(at 114.3 146.05 0)
 			(effects
@@
 			)
 		)
-		(property "URL" "https://www.digikey.com/en/products/detail/panasonic-electronic-components/ERJ-1GNF64R9C/2035977"
+		(property "URL" "https://www.digikey.com/en/products/detail/panasonic-electronic-components/ERA-3AEB151V/1465834"
 			(at 114.3 146.05 0)
 			(effects
@@
 		(on_board yes)
 		(dnp no)
-		(fields_autoplaced yes)
 		(property "Reference" "R4"
-			(at 114.3 144.78 90)
-			(effects
-				(font
-					(size 1.27 1.27)
-				)
-			)
-		)
-		(property "Value" "65"
-			(at 114.3 147.32 90)
+			(at 114.046 152.654 90)
+			(effects
+				(font
+					(size 1.27 1.27)
+				)
+			)
+		)
+		(property "Value" "85"
+			(at 114.046 154.686 90)
 			(effects
 				(font
@@
 			)
 		)
-		(property "Part Number" "ERJ-1GNF64R9C"
+		(property "Part Number" "ERJ-3EKF84R5V"
 			(at 114.3 151.13 0)
 			(effects
@@
 			)
 		)
-		(property "URL" "https://www.digikey.com/en/products/detail/panasonic-electronic-components/ERJ-1GNF64R9C/2035977"
+		(property "URL" "https://www.digikey.com/en/products/detail/panasonic-electronic-components/ERJ-3EKF84R5V/196495"
 			(at 114.3 151.13 0)
 			(effects

Commit message: pcb v1a
Parts:
- C13: footprint Capacitor_SMD:C_0402_1005Metric -> Capacitor_THT:C_Radial_D5.0mm_H5.0mm_P2.00mm
- C4: footprint Capacitor_SMD:C_0805_2012Metric -> Capacitor_THT:C_Radial_D5.0mm_H5.0mm_P2.00mm
- IC1: footprint digikey-footprints:SOIC-8_W5.3mm -> digikey-footprints:DIP-8_W7.62mm
- IC2: footprint AP7375-50SA-7 -> (none)
- R1, R2, R3, R4: footprint Resistor_SMD:R_0603_1608Metric -> Resistor_THT:R_Axial_DIN0204_L3.6mm_D1.6mm_P5.08mm_Horizontal
- TP3, TP4, TP5, TP6, TP7, TP8: footprint Connector_PinHeader_1.00mm:PinHeader_1x01_P1.00mm_Vertical -> Connector_PinHeader_2.54mm:PinHeader_1x01_P2.54mm_Vertical
Changed lines of the file:
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@@
 			)
 		)
-		(property "Footprint" "AP7375-50SA-7"
+		(property "Footprint" ""
 			(at 241.3 133.02 0)
 			(effects
@@
 			)
 		)
-		(property "Footprint" "Connector_PinHeader_1.00mm:PinHeader_1x01_P1.00mm_Vertical"
+		(property "Footprint" "Connector_PinHeader_2.54mm:PinHeader_1x01_P2.54mm_Vertical"
 			(at 208.28 105.41 0)
 			(effects
@@
 			)
 		)
-		(property "Footprint" "Connector_PinHeader_1.00mm:PinHeader_1x01_P1.00mm_Vertical"
+		(property "Footprint" "Connector_PinHeader_2.54mm:PinHeader_1x01_P2.54mm_Vertical"
 			(at 223.52 105.41 0)
 			(effects
@@
 			)
 		)
-		(property "Footprint" "Connector_PinHeader_1.00mm:PinHeader_1x01_P1.00mm_Vertical"
+		(property "Footprint" "Connector_PinHeader_2.54mm:PinHeader_1x01_P2.54mm_Vertical"
 			(at 262.89 105.41 0)
 			(effects
@@
 			)
 		)
-		(property "Footprint" "Connector_PinHeader_1.00mm:PinHeader_1x01_P1.00mm_Vertical"
+		(property "Footprint" "Connector_PinHeader_2.54mm:PinHeader_1x01_P2.54mm_Vertical"
 			(at 273.05 105.41 0)
 			(effects
@@
 			)
 		)
-		(property "Footprint" "Capacitor_SMD:C_0805_2012Metric"
+		(property "Footprint" "Capacitor_THT:C_Radial_D5.0mm_H5.0mm_P2.00mm"
 			(at 199.6948 43.18 0)
 			(effects
@@
 			)
 		)
-		(property "Footprint" "Connector_PinHeader_1.00mm:PinHeader_1x01_P1.00mm_Vertical"
+		(property "Footprint" "Connector_PinHeader_2.54mm:PinHeader_1x01_P2.54mm_Vertical"
 			(at 251.46 105.41 0)
 			(effects
@@
 			)
 		)
-		(property "Footprint" "Connector_PinHeader_1.00mm:PinHeader_1x01_P1.00mm_Vertical"
+		(property "Footprint" "Connector_PinHeader_2.54mm:PinHeader_1x01_P2.54mm_Vertical"
 			(at 237.49 105.41 0)
 			(effects
@@
 			)
 		)
-		(property "Footprint" "Capacitor_SMD:C_0402_1005Metric"
+		(property "Footprint" "Capacitor_THT:C_Radial_D5.0mm_H5.0mm_P2.00mm"
 			(at 260.6548 48.26 0)
 			(effects
@@
 			)
 		)
-		(property "Footprint" "Resistor_SMD:R_0603_1608Metric"
+		(property "Footprint" "Resistor_THT:R_Axial_DIN0204_L3.6mm_D1.6mm_P5.08mm_Horizontal"
 			(at 78.74 34.798 90)
 			(effects
@@
 			)
 		)
-		(property "Footprint" "Resistor_SMD:R_0603_1608Metric"
+		(property "Footprint" "Resistor_THT:R_Axial_DIN0204_L3.6mm_D1.6mm_P5.08mm_Horizontal"
 			(at 91.44 34.798 90)
 			(effects
@@
 			)
 		)
-		(property "Footprint" "Resistor_SMD:R_0603_1608Metric"
+		(property "Footprint" "Resistor_THT:R_Axial_DIN0204_L3.6mm_D1.6mm_P5.08mm_Horizontal"
 			(at 114.3 147.828 90)
 			(effects
@@
 			)
 		)
-		(property "Footprint" "digikey-footprints:SOIC-8_W5.3mm"
+		(property "Footprint" "digikey-footprints:DIP-8_W7.62mm"
 			(at 68.58 91.44 0)
 			(effects
@@
 			)
 		)
-		(property "Footprint" "Resistor_SMD:R_0603_1608Metric"
+		(property "Footprint" "Resistor_THT:R_Axial_DIN0204_L3.6mm_D1.6mm_P5.08mm_Horizontal"
 			(at 114.3 152.908 90)
 			(effects

Commit message: redesigning pcb to be smaller & use tag-connect
Parts:
- removed POT1: TC33X-2-103E, digikey-footprints:Trimpot_3.8mmx3.6mm_TC33X-2-103E, symbol dk_Trimmer-Potentiometers:TC33X-2-103E
- removed TP3: GND, Connector_PinHeader_2.54mm:PinHeader_1x01_P2.54mm_Vertical, symbol Connector:TestPoint
- removed TP4: 3V3, Connector_PinHeader_2.54mm:PinHeader_1x01_P2.54mm_Vertical, symbol Connector:TestPoint
- removed TP5: MISO, Connector_PinHeader_2.54mm:PinHeader_1x01_P2.54mm_Vertical, symbol Connector:TestPoint
- removed TP6: MOSI, Connector_PinHeader_2.54mm:PinHeader_1x01_P2.54mm_Vertical, symbol Connector:TestPoint
- removed TP7: SCK, Connector_PinHeader_2.54mm:PinHeader_1x01_P2.54mm_Vertical, symbol Connector:TestPoint
- removed TP8: RST, Connector_PinHeader_2.54mm:PinHeader_1x01_P2.54mm_Vertical, symbol Connector:TestPoint
- added J1: Conn_ARM_SWD_TagConnect_TC2030-NL, Connector:Tag-Connect_TC2030-IDC-NL_2x03_P1.27mm_Vertical, symbol Connector:Conn_ARM_SWD_TagConnect_TC2030-NL
- added S1: B3U-1000P, digikey-footprints:Switch_Tactile_SMD_B3U-1000P, symbol dk_Tactile-Switches:B3U-1000P
- C1: renamed from C4; footprint Capacitor_THT:C_Radial_D5.0mm_H5.0mm_P2.00mm -> Capacitor_SMD:C_0805_2012Metric
- C2: renamed from C13; footprint Capacitor_THT:C_Radial_D5.0mm_H5.0mm_P2.00mm -> Capacitor_SMD:C_0805_2012Metric
- IC1: footprint digikey-footprints:DIP-8_W7.62mm -> digikey-footprints:SOIC-8_W3.9mm
- IC2: footprint (none) -> Package_TO_SOT_SMD:TSOT-23
- R1, R2, R3, R4: footprint Resistor_THT:R_Axial_DIN0204_L3.6mm_D1.6mm_P5.08mm_Horizontal -> Resistor_SMD:R_0805_2012Metric
- TP1, TP2: footprint Connector_PinHeader_2.00mm:PinHeader_1x01_P2.00mm_Vertical -> Connector_PinHeader_2.54mm:PinHeader_1x01_P2.54mm_Vertical
Connections:
- net +5V: now also J1.1 (VCC)
- net DIM: now also S1.1
- net GND: now also D1.2 (K), J1.5 (GND), S1.2; no longer D1.3 (K)
- net MISO/G: now also J1.6 (SWO)
- net MOSI/R: now also J1.2 (SWDIO)
- net RST: now also J1.3 (~{RESET})
- net SCK/BATT: now also J1.4 (SWCLK)
- net G: now reaches R3.1
- net G: now also D1.3 (A2); no longer D1.1 (A1)
- net R: now reaches R4.1
- net R: now also D1.1 (A1); no longer D1.2 (A2)
Other:
- moved on the sheet: R3, R4

Commit message: pcb v1b, ready to manufacture
Parts:
- TP1, TP2: footprint Connector_PinHeader_2.54mm:PinHeader_1x01_P2.54mm_Vertical -> TestPoint:TestPoint_Pad_2.0x2.0mm
Changed lines of the file:
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@@
 			)
 		)
-		(property "Footprint" "Connector_PinHeader_2.54mm:PinHeader_1x01_P2.54mm_Vertical"
+		(property "Footprint" "TestPoint:TestPoint_Pad_2.0x2.0mm"
 			(at 139.7 67.31 0)
 			(effects
@@
 			)
 		)
-		(property "Footprint" "Connector_PinHeader_2.54mm:PinHeader_1x01_P2.54mm_Vertical"
+		(property "Footprint" "TestPoint:TestPoint_Pad_2.0x2.0mm"
 			(at 123.19 67.31 0)
 			(effects
